File: air-conditioner-board/air-conditioner-board.kicad_pcb (KiCad board)
At the start: 2 copper layers, 81.3 x 84.4 mm, 56 parts, among them Q1 BTA16-600BW, U1 DP1801B, U3 EL817, U4 MOC3021M

Commit message: Add layout version 2 - SMPS
Parts:
- removed J6, J7: ~, Connector_JOINT_TECH:TBG-5.0-KW-3P
- added H1: MountingHole, MountingHole:MountingHole_3.2mm_M3_Pad_Via, F.Cu at (57.7, 57.7)
- moved H3 72.1 mm to (128.0, 127.0)
- moved H4 56.8 mm to (128.0, 57.0)
- moved R15 43.7 mm to (96.5, 90.7), turned to 0 degrees
- moved J4 30.9 mm to (60.0, 73.0)
- moved BR2 30.3 mm to (87.5, 84.3), turned to 90 degrees
- moved C5 30.2 mm to (101.7, 116.8)
- moved C6 30.2 mm to (106.2, 116.8)
- moved PN1 30.2 mm to (119.2, 103.0)
- moved U2 30.2 mm to (131.2, 98.0)
- moved J5 29.1 mm to (125.0, 73.0)
- moved H2 28.5 mm to (56.4, 128.0)
- moved J3 27.6 mm to (116.0, 129.6)
- moved EC1 26.8 mm to (78.4, 94.4)
- moved BR1 26.8 mm to (76.4, 89.4)
- moved C1 26.8 mm to (59.3, 108.2)
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Routing:
- net NEUTRAL: track 165.2 -> 0.00 mm
- net /output/protection: track 126.1 -> 0.00 mm
- net +5V: track 118.5 -> 0.00 mm, vias 9 -> 12
- net ~230VAC: track 79.3 -> 0.00 mm
- net /output/sterowane wyjście: track 70.4 -> 0.00 mm
- net /MCU/enkoder A: track 53.4 -> 0.00 mm
- net /MCU/enkoder B: track 47.0 -> 0.00 mm
- net /MCU/potencjometr: track 44.8 -> 0.00 mm
- net /MCU/SDA: track 44.0 -> 0.00 mm
- net /MCU/SCL: track 36.3 -> 0.00 mm
- net Net-(Q1-G): track 28.0 -> 0.00 mm
- net /MCU/triac: track 20.0 -> 0.00 mm
- net /MCU/sine sinq: track 14.9 -> 0.00 mm
- net Net-(BR2--): track 11.8 -> 0.00 mm
- net /power/TR1 sec1: track 9.58 -> 0.00 mm
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- added copper zone on B.Cu, net /power/TR1 sec1
- added copper zone on B.Cu, net Net-(D2-Pad1)
- removed copper zone on F.Cu, net /output/sterowane wyjście
- removed copper zone on F.Cu, net GND
- removed copper zone on F.Cu, net ~230VAC
Other:
- board size 81.3 x 84.4 mm -> 85 x 85 mm

Commit message: Add layout version 2 complete
Parts:
- C5, C6: moved to F.Cu
- moved U3 14.2 mm to (125.8, 85.6), turned to -90 degrees
- moved BR2 6.72 mm to (92.2, 79.5), turned to -90 degrees
- moved C5 2.70 mm to (103.6, 118.7)
- moved C6 2.54 mm to (107.8, 118.7)
- moved U2 1.75 mm to (133.0, 98.0)
Connections:
- R13 pad 1: Net-(BR2--) -> Net-(BR2-+)
- R14 pad 1: Net-(BR2-+) -> Net-(BR2--)
- U3 pad 1: Net-(R14-Pad2) -> Net-(R13-Pad2)
- U3 pad 2: Net-(R13-Pad2) -> Net-(R14-Pad2)
Routing:
- net +5V: track 0.00 -> 104.4 mm
- net /output/protection: track 0.00 -> 85.8 mm
- net NEUTRAL: track 0.00 -> 81.9 mm
- net ~230VAC: track 0.00 -> 77.6 mm, vias 0 -> 9
- net /MCU/SDA: track 0.00 -> 51.7 mm
- net /MCU/SCL: track 0.00 -> 43.7 mm
- net /output/sterowane wyjście: track 0.00 -> 38.2 mm
- net Net-(Q1-G): track 0.00 -> 28.6 mm
- net /MCU/enkoder B: track 0.00 -> 23.5 mm
- net /MCU/sine sinq: track 0.00 -> 23.5 mm
- net /MCU/potencjometr: track 0.00 -> 20.4 mm
- net Net-(R13-Pad2): track 0.00 -> 18.6 mm
- net /MCU/enkoder A: track 0.00 -> 16.9 mm
- net Net-(R14-Pad2): track 0.00 -> 15.6 mm
- net Net-(BR2--): track 0.00 -> 10.8 mm
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- added copper zone on F.Cu, net GND
- added copper zone on B.Cu, net ~230VAC
- added copper zone on F.Cu, net ~230VAC

Commit message: final / production
Routing:
- net Net-(C4-Pad1): track 3.37 -> 0.00 mm
- net Net-(BR1--): track 7.28 -> 10.1 mm
- net GND: vias 66 -> 54
- added copper zone on B.Cu, net Net-(C4-Pad1)

Commit message: Add corrections
Parts:
- added R18: 1kΩ, Resistor_SMD:R_1206_3216Metric, B.Cu at (67.9, 121.7)
- moved C7 10.1 mm to (111.5, 118.2)
- moved HS1 7.55 mm to (92.5, 58.6)
- moved Q1 7.55 mm to (90.0, 62.8)
- moved JP1 2.75 mm to (69.7, 125.0)
- moved JP2 2.75 mm to (66.2, 125.0)
Connections:
- TR1 pad 1: /power/TR1 sec1 -> /power/TR1 sec2
- TR1 pad 2: /power/TR1 sec2 -> /power/TR1 sec1
Routing:
- net /power/TR1 sec1: track 0.00 -> 9.60 mm
- net /output/sterowane wyjście: track 38.2 -> 45.2 mm
- net +5V: track 104.4 -> 109.7 mm
- net ~230VAC: track 77.6 -> 72.3 mm
- net Net-(Q1-G): track 28.6 -> 32.8 mm
- net Net-(D3-K): track 3.23 -> 6.11 mm
- net /power/TR1 sec2: track 23.5 -> 24.8 mm
- net GND: vias 54 -> 17
