File: air-conditioner-board/air-conditioner-board.kicad_sch (KiCad schematic)
At the start: 4 parts

Commit message: Add layout version 2 - SMPS
Parts:
- added H1: MountingHole, MountingHole:MountingHole_3.2mm_M3_Pad_Via, symbol Mechanical:MountingHole
Other:
- moved on the sheet: PN1
Changed lines of the file:
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@@
+	(symbol
+		(lib_id "Mechanical:MountingHole")
+		(at 19.05 170.18 0)
+		(unit 1)
+		(exclude_from_sim no)
+		(in_bom no)
+		(on_board yes)
+		(dnp no)
+		(fields_autoplaced yes)
+		(property "Reference" "H1"
+			(at 21.59 168.9099 0)
+			(effects
+				(font
+					(size 1.27 1.27)
+				)
+				(justify left)
+			)
+		)
+		(property "Value" "MountingHole"
+			(at 21.59 171.4499 0)
+			(effects
+				(font
+					(size 1.27 1.27)
+				)
+				(justify left)
+			)
+		)
+		(property "Footprint" "MountingHole:MountingHole_3.2mm_M3_Pad_Via"
+			(at 19.05 170.18 0)
+			(effects
+				(font
+					(size 1.27 1.27)
+				)
+				(hide yes)
+			)
+		)
+		(property "Datasheet" "~"
+			(at 19.05 170.18 0)
+			(effects
+				(font
+					(size 1.27 1.27)
+				)
+				(hide yes)
+			)
+		)
+		(property "Description" "Mounting Hole without connection"
+			(at 19.05 170.18 0)
+			(effects
+				(font
+					(size 1.27 1.27)
+				)
+				(hide yes)
+			)
+		)
+		(instances
+			(project "air-conditioner-board"
+				(path "/e158d780-a4af-49fc-a6a2-d26b01f74f63"
+					(reference "H1")
+					(unit 1)
+				)
+			)
+		)
+	)
 	(symbol
 		(lib_id "Mechanical:MountingHole")
@@
 	(symbol
 		(lib_id "PCM_JLCPCB-Manufacturing:Part Number, PCM_JLCPCB, 0.8x0.15mm")
-		(at 17.78 171.45 0)
+		(at 17.78 166.37 0)
 		(unit 1)
 		(exclude_from_sim no)
@@
 		(fields_autoplaced yes)
 		(property "Reference" "PN1"
-			(at 19.05 170.8149 0)
+			(at 19.05 165.7349 0)
 			(effects
 				(font
@@
 		)
 		(property "Value" "~"
-			(at 19.05 172.72 0)
+			(at 19.05 167.64 0)
 			(effects
 				(font
@@
 		)
 		(property "Footprint" "PCM_JLCPCB:Part_Num_JLCPCB"
-			(at 17.78 171.45 0)
+			(at 17.78 166.37 0)
 			(effects
 				(font
@@
 		)
 		(property "Datasheet" "https://jlcpcb.com/help/article/How-to-remove-order-number-from-your-PCB"
-			(at 17.78 171.45 0)
+			(at 17.78 166.37 0)
 			(effects
 				(font
@@
 		)
 		(property "Description" "To indicate the location, simply add the text \"JLCJLCJLCJLC\" to the silk layer and select the \"Specify a location\" option when placing your order. Please note that if this option is not chosen, we may not notice that you have added the text.   Note: Use only \"JLCJLCJLCJLC\" without any additional characters. The font size should be larger than 0.8mm in height and 0.15mm in width."
-			(at 17.78 171.45 0)
-			(effects
-				(font
+			(at 17.78 166.37 0)
+			(effects
+				(font
