File: air-conditioner-board/power.kicad_sch (KiCad schematic)
At the start: 28 parts, among them U1 DP1801B

Commit message: Add corrections
Parts:
- added R18: 1kΩ, Resistor_SMD:R_1206_3216Metric, symbol Device:R
Connections:
- net TR1 sec1: now also TR1.2; no longer TR1.1
- net TR1 sec2: now also TR1.1, R18.2; no longer TR1.2
- net at C3.1, D3.1 (K), EC3.1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: now also R18.1
Other:
- moved on the sheet: EC3, JP1, JP2
